File: JLC_4layer_template/JLC_4layer_template.kicad_pcb (KiCad board)
At the start: 4 copper layers, 0 parts

Commit message: g
Other:
- rule solder_mask_min_width: 0.255 -> 0.25
Changed lines of the file:
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@@
     )
     (pad_to_mask_clearance 0)
-    (solder_mask_min_width 0.255)
+    (solder_mask_min_width 0.25)
     (pcbplotparams
       (layerselection 0x00010fc_ffffffff)
